Commit message: correct urdf

File: urdf/PhoXi3Dscanner.xacro (robot description, xacro)
@@ -5,6 +5,6 @@
     <xacro:PhoXi3Dscanner scanner_parent = "base_link" scanner_name = "PhoXi3Dscanner" sensor_parent = "PhoXi3Dscanner" sensor_name = "PhoXi3Dscanner_sensor" >
         <origin xyz="0 0 0" rpy="0 0 0" /> <!--PhoXi3Dscanner origin-->
-        <xacro:PhoXi3DscannerM_default_sensor_origin /> <!--Extrinsic calibration data-->
-        <xacro:PhoXi3DscannerM_meshes /> <!--meshes-->
+        <xacro:PhoXi3DscannerS_default_sensor_origin /> <!--Extrinsic calibration data-->
+        <xacro:PhoXi3DscannerS_meshes /> <!--meshes-->
     </xacro:PhoXi3Dscanner>
     <link name ="base_link"/>

File: urdf/PhoXi3Dscanner_values.xacro (robot description, xacro)
@@ -11,5 +11,5 @@
     <!--PhoXi3Dscanner S-->
     <xacro:macro name="PhoXi3DscannerS_default_sensor_origin">
-        <origin xyz="${0.23 / 2.0} 0.0168 0.035" rpy="0 -0.26965337 0" />
+        <origin xyz="${-0.23 / 2.0} 0.0168 0.035" rpy="0 -0.26965337 ${pi}" />
     </xacro:macro>
     <xacro:macro name="PhoXi3DscannerS_meshes">

Commit message: update urdf

File: urdf/PhoXi3Dscanner.xacro (robot description, xacro)
@@ -3,5 +3,5 @@
     <xacro:include filename="$(find phoxi_camera)/urdf/PhoXi3Dscanner_values.xacro"/> <!--Scanner values-->
     <xacro:include filename="$(find phoxi_camera)/urdf/PhoXi3Dscanner_macro.xacro"/>  <!--Scanner macro-->
-    <xacro:PhoXi3Dscanner scanner_parent = "base_link" scanner_name = "PhoXi3Dscanner" sensor_parent = "PhoXi3Dscanner" sensor_name = "PhoXi3Dscanner_sensor" >
+    <xacro:PhoXi3Dscanner scanner_name = "PhoXi3Dscanner" sensor_parent = "base_link" sensor_name = "PhoXi3Dscanner_sensor" >
         <origin xyz="0 0 0" rpy="0 0 0" /> <!--PhoXi3Dscanner origin-->
         <xacro:PhoXi3DscannerS_default_sensor_origin /> <!--Extrinsic calibration data-->

File: urdf/PhoXi3Dscanner_macro.xacro (robot description, xacro)
@@ -1,13 +1,13 @@
 <?xml version="1.0" ?>
 <robot xmlns:xacro="http://ros.org/wiki/xacro">
-    <xacro:macro name = "PhoXi3Dscanner" params ="scanner_parent scanner_name *scanner_origin sensor_parent sensor_name *sensor_origin *visual *collision">
-        <joint name="${scanner_parent}_to_${scanner_name}_joint" type="fixed">
-            <parent link="${scanner_parent}"/>
-            <child link="${scanner_name}"/>
-            <xacro:insert_block name="scanner_origin" />
-        </joint>
+    <xacro:macro name = "PhoXi3Dscanner" params ="scanner_name *scanner_origin sensor_parent sensor_name *sensor_origin *visual *collision">
         <joint name="${sensor_parent}_to_${sensor_name}_joint" type="fixed">
             <parent link="${sensor_parent}"/>
             <child link="${sensor_name}"/>
+            <xacro:insert_block name="scanner_origin" />
+        </joint>
+        <joint name="${sensor_name}_to_${scanner_name}_joint" type="fixed">
+            <parent link="${sensor_name}"/>
+            <child link="${scanner_name}"/>
             <xacro:insert_block name="sensor_origin" />
         </joint>
